Commit message: Update description

File: src/description/description/robot.urdf.xacro (robot description, xacro)
@@ -2,4 +2,6 @@
 <!-- add xmlns:macro="link" to use xacro extension -->
 <robot name="robot" xmlns:xacro="http://www.ros.org/wiki/xacro">
+    <!-- Include -->
+    <xacro:include filename="inertials.xacro" />
     <!-- Define constant variables using xacro -->
     <xacro:property name="base_length" value="0.2" />
@@ -8,4 +10,5 @@
     <xacro:property name="wheel_radius" value="0.045" />
     <xacro:property name="wheel_length" value="0.01" />
+    <xacro:property name="robot_namespace" value="/ackrobot"/>
     <material name="red">
         <color rgba="1 0 0 1"/>
@@ -17,14 +20,33 @@
         <color rgba="0.5 0.5 0.5 1" />
     </material>
-    <link name="footprint_link" />
+    <material name="invisible">
+        <color rgba="0.0 0.0 0.0 0.0"/>
+    </material>
+    <link name="base_footprint" />
     <link name="base_link">
         <visual>
             <geometry>
-                <box size="${base_length} ${base_width} ${base_height}" />
+                <box size="${base_length} ${base_width} ${base_height - (wheel_radius / 2)}" />
             </geometry>
             <origin xyz="0 0 ${base_height / 2.0}" rpy="0 0 0" />
             <material name="red" />
         </visual>
+        <xacro:inertial_box mass="3.0" x="${base_length}" y="${base_width}" z="${base_height - (wheel_radius / 2)}">
+            <origin xyz="0 0 ${base_height / 2.0}" rpy="0 0 0"/>
+        </xacro:inertial_box>
     </link>
+    <gazebo reference="base_link">
+        <!--Stiffness -->
+        <kp>1000000.0</kp>
+        <!--Dampening-->
+        <kd>0.1</kd>
+        <dampingFactor>0</dampingFactor>
+        <material>Gazebo/Red</material>
+        <selfCollide>true</selfCollide>
+        <turnGravityOff>false</turnGravityOff>
+        <mu1 value="0.1"/>
+        <mu2 value="0.1"/>
+        <fdir1 value="0 0 0"/>
+    </gazebo>
     <!-- Back Right Wheel -->
     <link name="back_right_wheel_link">
@@ -44,5 +66,5 @@
             </geometry>
             <origin xyz="0 0 0" rpy="${pi / 2.0} 0 0" />
-            <material name="grey" />
+            <material name="orange" />
         </visual>
     </link>
@@ -64,10 +86,20 @@
             </geometry>
             <origin xyz="0 0 0" rpy="${pi / 2.0} 0 0" />
-            <material name="grey" />
+            <material name="orange" />
         </visual>
+    </link>
+    <!-- Virtual Front Wheel -->
+    <link name="virtual_front_wheel">
+      <visual>
+        <origin xyz="0 0 0" rpy="${pi/2} 0 ${pi/2}"/>
+        <geometry>
+          <cylinder length="0.01" radius="${wheel_radius}"/>
+        </geometry>
+        <material name="invisible"/>
+      </visual>
     </link>
     <!-- Joints -->
     <joint name="footprint_base_joint" type="fixed">
-        <parent link="footprint_link" />
+        <parent link="base_footprint" />
         <child link="base_link" />
         <origin xyz="0 0 ${wheel_radius}" rpy="0 0 0" />
@@ -77,5 +109,5 @@
         <parent link="base_link" />
         <child link="back_right_wheel_link" />
-        <origin xyz="${-base_length / 4.0} ${-(base_width + wheel_length) / 2.0} 0" rpy="0 0 0" />
+        <origin xyz="${-base_length / 2.0} ${-(base_width + wheel_length) / 2.0} 0" rpy="0 0 0" />
         <axis xyz="0 1 0" />
     </joint>
@@ -83,18 +115,34 @@
         <parent link="base_link" />
         <child link="back_left_wheel_link" />
-        <origin xyz="${-base_length / 4.0} ${(base_width + wheel_length) / 2.0} 0" rpy="0 0 0" />
+        <origin xyz="${-base_length / 2.0} ${(base_width + wheel_length) / 2.0} 0" rpy="0 0 0" />
         <axis xyz="0 1 0" />
     </joint>
     <joint name="base_front_right_wheel_joint" type="continuous">
-        <parent link="base_link" />
+        <parent link="virtual_front_wheel" />
         <child link="front_right_wheel_link" />
-        <origin xyz="${base_length / 4.0} ${-(base_width + wheel_length) / 2.0} 0" rpy="0 0 0" />
+        <origin xyz="0 ${-(base_width + wheel_length) / 2.0} 0" rpy="0 0 0" />
         <axis xyz="0 1 0" />
     </joint>
     <joint name="base_front_left_wheel_joint" type="continuous">
-        <parent link="base_link" />
+        <parent link="virtual_front_wheel" />
         <child link="front_left_wheel_link" />
-        <origin xyz="${base_length / 4.0} ${(base_width + wheel_length) / 2.0} 0" rpy="0 0 0" />
+        <origin xyz="0 ${(base_width + wheel_length) / 2.0} 0" rpy="0 0 0" />
         <axis xyz="0 1 0" />
     </joint>
+    <joint name="virtual_front_wheel_joint" type="revolute">
+      <parent link="base_link"/>
+      <child link="virtual_front_wheel"/>
+      <origin xyz="${base_length/2} 0 0" rpy="0 0 0"/>
+      <axis xyz="0 0 1"/>
+      <limit lower="-0.4" upper="0.4" effort="100.0" velocity="0.0"/>
+      <dynamics damping="0.2"/>
+    </joint>
+    <!-- Gazebo plugins -->
+    <gazebo>
+        <plugin name="gazebo_ros_control" filename="libgazebo_ros_control.so">
+        <robotNamespace>${robot_namespace}</robotNamespace>
+        <robotSimType>steer_bot_hardware_gazebo/SteerBotHardwareGazebo</robotSimType>
+        <legacyModeNS>false</legacyModeNS>
+        </plugin>
+    </gazebo>
 </robot>

Commit message: Caught Bug on Gazebo

File: src/description/description/robot.urdf.xacro (robot description, xacro)
@@ -1,148 +1,5 @@
 <?xml version="1.0"?>
-<!-- add xmlns:macro="link" to use xacro extension -->
-<robot name="robot" xmlns:xacro="http://www.ros.org/wiki/xacro">
-    <!-- Include -->
-    <xacro:include filename="inertials.xacro" />
-    <!-- Define constant variables using xacro -->
-    <xacro:property name="base_length" value="0.2" />
-    <xacro:property name="base_width" value="0.13" />
-    <xacro:property name="base_height" value="0.1" />
-    <xacro:property name="wheel_radius" value="0.045" />
-    <xacro:property name="wheel_length" value="0.01" />
-    <xacro:property name="robot_namespace" value="/ackrobot"/>
-    <material name="red">
-        <color rgba="1 0 0 1"/>
-    </material>
-    <material name="orange">
-        <color rgba="1 0.6 0 1" />
-    </material>
-    <material name="grey">
-        <color rgba="0.5 0.5 0.5 1" />
-    </material>
-    <material name="invisible">
-        <color rgba="0.0 0.0 0.0 0.0"/>
-    </material>
-    <link name="base_footprint" />
-    <link name="base_link">
-        <visual>
-            <geometry>
-                <box size="${base_length} ${base_width} ${base_height - (wheel_radius / 2)}" />
-            </geometry>
-            <origin xyz="0 0 ${base_height / 2.0}" rpy="0 0 0" />
-            <material name="red" />
-        </visual>
-        <xacro:inertial_box mass="3.0" x="${base_length}" y="${base_width}" z="${base_height - (wheel_radius / 2)}">
-            <origin xyz="0 0 ${base_height / 2.0}" rpy="0 0 0"/>
-        </xacro:inertial_box>
-    </link>
-    <gazebo reference="base_link">
-        <!--Stiffness -->
-        <kp>1000000.0</kp>
-        <!--Dampening-->
-        <kd>0.1</kd>
-        <dampingFactor>0</dampingFactor>
-        <material>Gazebo/Red</material>
-        <selfCollide>true</selfCollide>
-        <turnGravityOff>false</turnGravityOff>
-        <mu1 value="0.1"/>
-        <mu2 value="0.1"/>
-        <fdir1 value="0 0 0"/>
-    </gazebo>
-    <!-- Back Right Wheel -->
-    <link name="back_right_wheel_link">
-        <visual>
-            <geometry>
-                <cylinder radius="${wheel_radius}" length="${wheel_length}" />
-            </geometry>
-            <origin xyz="0 0 0" rpy="${pi / 2.0} 0 0" />
-            <material name="orange" />
-        </visual>
-    </link>
-    <!-- Back Left Wheel -->
-    <link name="back_left_wheel_link">
-        <visual>
-            <geometry>
-                <cylinder radius="${wheel_radius}" length="${wheel_length}" />
-            </geometry>
-            <origin xyz="0 0 0" rpy="${pi / 2.0} 0 0" />
-            <material name="orange" />
-        </visual>
-    </link>
-    <!-- Front Right Wheel -->
-    <link name="front_right_wheel_link">
-        <visual>
-            <geometry>
-                <cylinder radius="${wheel_radius}" length="${wheel_length}" />
-            </geometry>
-            <origin xyz="0 0 0" rpy="${pi / 2.0} 0 0" />
-            <material name="orange" />
-        </visual>
-    </link>
-    <!-- Front Left Wheel -->
-    <link name="front_left_wheel_link">
-        <visual>
-            <geometry>
-                <cylinder radius="${wheel_radius}" length="${wheel_length}" />
-            </geometry>
-            <origin xyz="0 0 0" rpy="${pi / 2.0} 0 0" />
-            <material name="orange" />
-        </visual>
-    </link>
-    <!-- Virtual Front Wheel -->
-    <link name="virtual_front_wheel">
-      <visual>
-        <origin xyz="0 0 0" rpy="${pi/2} 0 ${pi/2}"/>
-        <geometry>
-          <cylinder length="0.01" radius="${wheel_radius}"/>
-        </geometry>
-        <material name="invisible"/>
-      </visual>
-    </link>
-    <!-- Joints -->
-    <joint name="footprint_base_joint" type="fixed">
-        <parent link="base_footprint" />
-        <child link="base_link" />
-        <origin xyz="0 0 ${wheel_radius}" rpy="0 0 0" />
-        <axis xyz="0 0 0" />
-    </joint>
-    <joint name="base_back_right_wheel_joint" type="continuous">
-        <parent link="base_link" />
-        <child link="back_right_wheel_link" />
-        <origin xyz="${-base_length / 2.0} ${-(base_width + wheel_length) / 2.0} 0" rpy="0 0 0" />
-        <axis xyz="0 1 0" />
-    </joint>
-    <joint name="base_back_left_wheel_joint" type="continuous">
-        <parent link="base_link" />
-        <child link="back_left_wheel_link" />
-        <origin xyz="${-base_length / 2.0} ${(base_width + wheel_length) / 2.0} 0" rpy="0 0 0" />
-        <axis xyz="0 1 0" />
-    </joint>
-    <joint name="base_front_right_wheel_joint" type="continuous">
-        <parent link="virtual_front_wheel" />
-        <child link="front_right_wheel_link" />
-        <origin xyz="0 ${-(base_width + wheel_length) / 2.0} 0" rpy="0 0 0" />
-        <axis xyz="0 1 0" />
-    </joint>
-    <joint name="base_front_left_wheel_joint" type="continuous">
-        <parent link="virtual_front_wheel" />
-        <child link="front_left_wheel_link" />
-        <origin xyz="0 ${(base_width + wheel_length) / 2.0} 0" rpy="0 0 0" />
-        <axis xyz="0 1 0" />
-    </joint>
-    <joint name="virtual_front_wheel_joint" type="revolute">
-      <parent link="base_link"/>
-      <child link="virtual_front_wheel"/>
-      <origin xyz="${base_length/2} 0 0" rpy="0 0 0"/>
-      <axis xyz="0 0 1"/>
-      <limit lower="-0.4" upper="0.4" effort="100.0" velocity="0.0"/>
-      <dynamics damping="0.2"/>
-    </joint>
-    <!-- Gazebo plugins -->
-    <gazebo>
-        <plugin name="gazebo_ros_control" filename="libgazebo_ros_control.so">
-        <robotNamespace>${robot_namespace}</robotNamespace>
-        <robotSimType>steer_bot_hardware_gazebo/SteerBotHardwareGazebo</robotSimType>
-        <legacyModeNS>false</legacyModeNS>
-        </plugin>
-    </gazebo>
+<robot xmlns:xacro="http://www.ros.org/wiki/xacro"  name="ackrobot">
+    <xacro:include filename="robot_core.urdf.xacro"/>
+    <xacro:include filename="gazebo_control.xacro"/>
 </robot>
