Commit message: Update description

File: src/description/description/gazebo_control.xacro (robot description, xacro)
@@ -14,6 +14,6 @@
                 <param name="min">-0.4</param>
                 <param name="max">0.4</param>
-              </command_interface>
-              <state_interface name="position">
+            </command_interface>
+              <!-- <state_interface name="position">
                 <param name="initial_value">0.0</param>
               </state_interface>
@@ -21,5 +21,5 @@
                 <param name="initial_value">0.0</param>
               </state_interface>
-              <state_interface name="effort"/>
+              <state_interface name="effort"/> -->
         </joint>
         <joint name="virtual_rear_wheel_joint">
@@ -28,11 +28,11 @@
                 <param name="max">5</param>
               </command_interface>
-              <state_interface name="position">
-                <param name="initial_value">0.0</param>
-              </state_interface>
-              <state_interface name="velocity">
-                <param name="initial_value">0.0</param>
-              </state_interface>
-              <state_interface name="effort"/>
+                <!-- <state_interface name="position">
+                  <param name="initial_value">0.0</param>
+                </state_interface>
+                <state_interface name="velocity">
+                  <param name="initial_value">0.0</param>
+                </state_interface>
+                <state_interface name="effort"/> -->
         </joint>
     </ros2_control>
@@ -82,3 +82,19 @@
       <material>Gazebo/Orange</material>
     </gazebo>
+    <gazebo reference="virtual_front_wheel_joint">
+      <!-- <mu1 value="2.0"/>
+      <mu2 value="2.0"/>
+      <kp  value="10000000.0" />
+      <kd  value="1.0" />
+      <fdir1 value="0 1 0"/>  -->
+      <material>Gazebo/Invisible</material>
+    </gazebo>
+    <gazebo reference="virtual_rear_wheel_joint">
+      <!-- <mu1 value="2.0"/>
+      <mu2 value="2.0"/>
+      <kp  value="10000000.0" />
+      <kd  value="1.0" />
+      <fdir1 value="0 1 0"/>  -->
+      <material>Gazebo/Invisible</material>
+    </gazebo>
 </robot>

Commit message: Update Description

File: src/description/description/gazebo_control.xacro (robot description, xacro)
@@ -88,5 +88,5 @@
       <kd  value="1.0" />
       <fdir1 value="0 1 0"/>  -->
-      <material>Gazebo/Invisible</material>
+      <material>Gazebo/Red</material>
     </gazebo>
     <gazebo reference="virtual_rear_wheel_joint">
@@ -96,5 +96,5 @@
       <kd  value="1.0" />
       <fdir1 value="0 1 0"/>  -->
-      <material>Gazebo/Invisible</material>
+      <material>Gazebo/Red</material>
     </gazebo>
 </robot>

File: src/description/description/robot_core.urdf.xacro (robot description, xacro)
@@ -77,7 +77,4 @@
             <material name="orange" />
         </visual>
-        <xacro:inertial_cylinder mass="0.25" length="${wheel_length}" radius="${wheel_radius}">
-            <origin xyz="0 0 0" rpy="${pi / 2.0} 0 0"/>
-        </xacro:inertial_cylinder>
     </link>
     <!-- Virtual Rear Wheel -->
@@ -131,11 +128,14 @@
     <!-- Virtual Front Wheel -->
     <link name="virtual_front_wheel">
-      <visual>
-        <origin xyz="0 0 0" rpy="${pi/2} 0 ${pi/2}"/>
-        <geometry>
-          <cylinder length="0.01" radius="${wheel_radius}"/>
-        </geometry>
-        <material name="invisible"/>
-      </visual>
+        <visual>
+            <origin xyz="0 0 0" rpy="${pi/2} 0 ${pi/2}"/>
+            <geometry>
+            <cylinder length="0.01" radius="${wheel_radius}"/>
+            </geometry>
+            <material name="invisible"/>
+        </visual>
+        <xacro:inertial_cylinder mass="0.0000001" length="0.01" radius="${wheel_radius}">
+            <origin xyz="0 0 0" rpy="${pi / 2.0} 0 ${pi / 2.0}"/>
+        </xacro:inertial_cylinder>
     </link>
     <!-- Joints -->
@@ -145,40 +145,4 @@
         <origin xyz="0 0 ${wheel_radius}" rpy="0 0 0" />
         <axis xyz="0 0 0" />
-    </joint>
-    <joint name="base_rear_right_wheel_joint" type="continuous">
-        <parent link="chassis" />
-        <child link="rear_right_wheel_link" />
-        <origin xyz="${-base_length / 2.0} ${-(base_width + wheel_length) / 2.0} 0" rpy="0 0 0" />
-        <axis xyz="0 1 0" />
-        <limit effort="100.0" velocity="100.0"/>
-        <dynamics damping="0.2"/>
-        <mimic joint="virtual_rear_wheel_joint" multiplier="1.0" offset="0.0"/>
-    </joint>
-    <joint name="base_rear_left_wheel_joint" type="continuous">
-        <parent link="chassis" />
-        <child link="rear_left_wheel_link" />
-        <origin xyz="${-base_length / 2.0} ${(base_width + wheel_length) / 2.0} 0" rpy="0 0 0" />
-        <axis xyz="0 1 0" />
-        <limit effort="100.0" velocity="100.0"/>
-        <dynamics damping="0.2"/>
-        <mimic joint="virtual_rear_wheel_joint" multiplier="1.0" offset="0.0"/>
-    </joint>
-    <joint name="base_front_right_wheel_joint" type="continuous">
-        <parent link="chassis" />
-        <child link="front_right_wheel_link" />
-        <origin xyz="${base_length/2} ${-(base_width + wheel_length) / 2.0} 0" rpy="0 0 0" />
-        <axis xyz="0 0   1" />
-        <limit lower="-0.4" upper="0.4" effort="100.0" velocity="0.0"/>
-        <dynamics damping="0.2"/>
-        <mimic joint="virtual_front_wheel_joint" multiplier="1.0" offset="0.0"/>
-    </joint>
-    <joint name="base_front_left_wheel_joint" type="continuous">
-        <parent link="chassis" />
-        <child link="front_left_wheel_link" />
-        <origin xyz="${base_length/2} ${(base_width + wheel_length) / 2.0} 0" rpy="0 0 0" />
-        <axis xyz="0 0 1" />
-        <limit lower="-0.4" upper="0.4" effort="100.0" velocity="0.0"/>
-        <dynamics damping="0.2"/>
-        <mimic joint="virtual_front_wheel_joint" multiplier="1.0" offset="0.0"/>
     </joint>
     <joint name="virtual_front_wheel_joint" type="revolute">
@@ -189,4 +153,7 @@
       <limit lower="-0.4" upper="0.4" effort="100.0" velocity="0.0"/>
       <dynamics damping="0.2"/>
+        <gazebo>
+            <disable_physics>true</disable_physics>
+        </gazebo>
     </joint>
     <joint name="virtual_rear_wheel_joint" type="continuous">
@@ -197,4 +164,63 @@
       <limit effort="100.0" velocity="100.0"/>
       <dynamics damping="0.2"/>
-    </joint>
+        <gazebo>
+            <disable_physics>true</disable_physics>
+        </gazebo>
+    </joint>
+    <joint name="base_rear_right_wheel_joint" type="continuous">
+        <parent link="chassis" />
+        <child link="rear_right_wheel_link" />
+        <origin xyz="${-base_length / 2.0} ${-(base_width + wheel_length) / 2.0} 0" rpy="0 0 0" />
+        <axis xyz="0 1 0" />
+        <limit effort="100.0" velocity="100.0"/>
+        <dynamics damping="0.2"/>
+        <mimic joint="virtual_rear_wheel_joint" multiplier="1.0" offset="0.0"/>
+    </joint>
+    <joint name="base_rear_left_wheel_joint" type="continuous">
+        <parent link="chassis" />
+        <child link="rear_left_wheel_link" />
+        <origin xyz="${-base_length / 2.0} ${(base_width + wheel_length) / 2.0} 0" rpy="0 0 0" />
+        <axis xyz="0 1 0" />
+        <limit effort="100.0" velocity="100.0"/>
+        <dynamics damping="0.2"/>
+        <mimic joint="virtual_rear_wheel_joint" multiplier="1.0" offset="0.0"/>
+    </joint>
+    <joint name="base_front_right_wheel_joint" type="continuous">
+        <parent link="chassis" />
+        <child link="front_right_wheel_link" />
+        <origin xyz="${base_length/2} ${-(base_width + wheel_length) / 2.0} 0" rpy="0 0 0" />
+        <axis xyz="0 0   1" />
+        <limit lower="-0.4" upper="0.4" effort="100.0" velocity="0.0"/>
+        <dynamics damping="0.2"/>
+        <mimic joint="virtual_front_wheel_joint" multiplier="1.0" offset="0.0"/>
+    </joint>
+    <joint name="base_front_left_wheel_joint" type="continuous">
+        <parent link="chassis" />
+        <child link="front_left_wheel_link" />
+        <origin xyz="${base_length/2} ${(base_width + wheel_length) / 2.0} 0" rpy="0 0 0" />
+        <axis xyz="0 0 1" />
+        <limit lower="-0.4" upper="0.4" effort="100.0" velocity="0.0"/>
+        <dynamics damping="0.2"/>
+        <mimic joint="virtual_front_wheel_joint" multiplier="1.0" offset="0.0"/>
+    </joint>
+    <!-- <transmission name="virtual_front_wheel_joint_trans">
+      <type>transmission_interface/SimpleTransmission</type>
+      <actuator name="virtual_front_wheel_joint_motor">
+        <mechanicalReduction>1</mechanicalReduction>
+        <hardwareInterface>hardware_interface/PositionJointInterface</hardwareInterface>
+      </actuator>
+      <joint name="virtual_front_wheel_joint">
+        <hardwareInterface>hardware_interface/PositionJointInterface</hardwareInterface>
+      </joint>
+    </transmission>
+    <transmission name="virtual_rear_wheel_joint_trans">
+      <type>transmission_interface/SimpleTransmission</type>
+      <actuator name="virtual_rear_wheel_joint_motor">
+        <mechanicalReduction>1</mechanicalReduction>
+        <hardwareInterface>hardware_interface/VelocityJointInterface</hardwareInterface>
+      </actuator>
+      <joint name="virtual_rear_wheel_joint">
+        <hardwareInterface>hardware_interface/VelocityJointInterface</hardwareInterface>
+      </joint>
+    </transmission> -->
 </robot>
