Commit message: Update Validate

File: src/ack_description/urdf/gazebo.xacro (robot description, xacro)
@@ -1,4 +1,4 @@
 <?xml version="1.0"?>
-<robot xmlns:xacro="http://www.ros.org/wiki/xacro" name="example">
+<robot xmlns:xacro="http://www.ros.org/wiki/xacro" name="ackbot">
     <xacro:include filename="inertial_macros.xacro"/>
     <ros2_control name="GazeboSystem" type="system">
@@ -6,5 +6,5 @@
             <plugin>gazebo_ros2_control/GazeboSystem</plugin>
         </hardware>
-        <joint name="left_joint_b">
+        <joint name="left_rear_wheel">
             <command_interface name="velocity"/>
             <state_interface name="position">
@@ -14,5 +14,5 @@
             <state_interface name="effort"/>
         </joint>
-        <joint name="right_joint_b">
+        <joint name="right_rear_wheel">
             <command_interface name="velocity"/>
             <state_interface name="position">
@@ -22,21 +22,5 @@
             <state_interface name="effort"/>
         </joint>
-        <joint name="left_joint_f">
-            <command_interface name="velocity"/>
-            <state_interface name="position">
-                <param name="initial_value">0.0</param>
-            </state_interface>
-            <state_interface name="velocity"/>
-            <state_interface name="effort"/>
-        </joint>
-        <joint name="right_joint_f">
-            <command_interface name="velocity"/>
-            <state_interface name="position">
-                <param name="initial_value">0.0</param>
-            </state_interface>
-            <state_interface name="velocity"/>
-            <state_interface name="effort"/>
-        </joint>
-        <joint name="left_joint_s">
+        <joint name="left_steer">
             <command_interface name="position">
                 <param name="min">-0.60</param>
@@ -50,5 +34,5 @@
             <state_interface name="effort"/>
         </joint>
-        <joint name="right_joint_s">
+        <joint name="right_steer">
             <command_interface name="position">
                 <param name="min">-0.60</param>
@@ -69,38 +53,55 @@
         </plugin>
     </gazebo>
+    <gazebo>
+      <plugin name="ground_truth_controller" filename="libgazebo_ros_p3d.so">
+        <ros>
+          <namespace>/ground_truth</namespace>
+          <remapping>odom:=pose</remapping>
+        </ros>
+        <body_name>base_link</body_name>
+        <frameName>world</frameName>
+        <updateRate>100.0</updateRate>
+      </plugin>
+    </gazebo>
+    <!-- <gazebo>
+        <plugin name="gazebo_ros_joint_state_publisher" filename="libgazebo_ros_joint_state_publisher.so">
+            <always_on>true</always_on>
+            <update_rate>100.0</update_rate>
+        </plugin>
+    </gazebo> -->
     <gazebo reference="chassis">
-        <mu1>0.2</mu1>
-        <mu2>0.2</mu2>
-        <material>Gazebo/Green</material>
-    </gazebo>
-    <gazebo reference="left_steer">
-        <mu1>0.2</mu1>
-        <mu2>0.2</mu2>
-        <material>Gazebo/Green</material>
-    </gazebo>
-    <gazebo reference="right_steer">
-        <mu1>0.2</mu1>
-        <mu2>0.2</mu2>
-        <material>Gazebo/Green</material>
-    </gazebo>
-    <gazebo reference="left_wheel_f">
         <mu1>0.2</mu1>
         <mu2>0.2</mu2>
         <material>Gazebo/Red</material>
     </gazebo>
-    <gazebo reference="left_wheel_b">
+    <gazebo reference="left_steer_link">
         <mu1>0.2</mu1>
         <mu2>0.2</mu2>
         <material>Gazebo/Red</material>
     </gazebo>
-    <gazebo reference="right_wheel_f">
+    <gazebo reference="right_steer_link">
         <mu1>0.2</mu1>
         <mu2>0.2</mu2>
-        <material>Gazebo/Blue</material>
+        <material>Gazebo/Red</material>
     </gazebo>
-    <gazebo reference="right_wheel_b">
+    <gazebo reference="left_front_wheel_link">
         <mu1>0.2</mu1>
         <mu2>0.2</mu2>
-        <material>Gazebo/Blue</material>
+        <material>Gazebo/Black</material>
+    </gazebo>
+    <gazebo reference="left_rear_wheel_link">
+        <mu1>0.2</mu1>
+        <mu2>0.2</mu2>
+        <material>Gazebo/Black</material>
+    </gazebo>
+    <gazebo reference="right_front_wheel_link">
+        <mu1>0.2</mu1>
+        <mu2>0.2</mu2>
+        <material>Gazebo/Black</material>
+    </gazebo>
+    <gazebo reference="right_rear_wheel_link">
+        <mu1>0.2</mu1>
+        <mu2>0.2</mu2>
+        <material>Gazebo/Black</material>
     </gazebo>
 </robot>

File: src/ack_description/urdf/imu.xacro (robot description, xacro)
@@ -11,5 +11,7 @@
                 <cylinder radius="0.02" length="0.01"/>
             </geometry>
-            <material name="red"/>
+            <material name="Yellow">
+                <color rgba="1 1 0 1"/>
+            </material>
         </visual>
         <collision>

File: src/ack_description/urdf/robot.xacro (robot description, xacro)
@@ -1,6 +1,7 @@
 <?xml version="1.0"?>
-<robot xmlns:xacro="http://www.ros.org/wiki/xacro" name="robot">
+<robot xmlns:xacro="http://www.ros.org/wiki/xacro" name="ackbot">
     <xacro:include filename="gazebo.xacro"/>
     <xacro:include filename="imu.xacro"/>
+    <xacro:include filename="transmission.xacro"/>
     <!-- BASE LINK -->
     <link name="base_link">
@@ -13,95 +14,119 @@
     </joint>
     <link name="chassis">
-        <xacro:inertial_box mass="3" x="0.2" y="0.13" z="0.1">
-            <origin xyz="0 0 0.005" rpy="0 0 0"/>
+        <xacro:inertial_box mass="3" x="0.2" y="0.13" z="0.06">
+            <origin xyz="0 0 0.025" rpy="0 0 0"/>
         </xacro:inertial_box>
         <visual>
-            <origin xyz="0 0 0" rpy="0 0 0" />
-            <geometry>
-                <mesh filename="file:///$(find ack_description)/meshes/Body.STL"/>
-            </geometry>
-        </visual>
-        <collision>
-            <origin xyz="0 0 0" rpy="0 0 0" />
-            <geometry>
-                <mesh filename="file:///$(find ack_description)/meshes/Body.STL"/>
+            <origin xyz="0 0 0.025" rpy="0 0 0" />
+            <geometry>
+                <!-- <mesh filename="file:///$(find ack_description)/meshes/Body.STL"/> -->
+                <box size="0.2 0.13 0.05"/>
+            </geometry>
+            <material name="Red">
+                <color rgba="1 0 0 1"/>
+            </material>
+        </visual>
+        <collision>
+            <origin xyz="0 0 0.025" rpy="0 0 0" />
+            <geometry>
+                <box size="0.2 0.13 0.06"/>
             </geometry>
         </collision>
     </link>
     <!-- WHEEL LINK -->
-    <link name="right_wheel_b">
-        <xacro:inertial_cylinder mass="0.1" length="0.01" radius="0.045">
-            <origin xyz="0 0 0" rpy="0 0 0"/>
-        </xacro:inertial_cylinder>
-        <visual>
-            <origin xyz="0 0 0" rpy="0 0 0" />
-            <geometry>
-                <mesh filename="file:///$(find ack_description)/meshes/Wheel.STL" />
-            </geometry>
-        </visual>
-        <collision>
-            <origin xyz="0 0 0" rpy="0 0 0" />
-            <geometry>
-                <mesh filename="file:///$(find ack_description)/meshes/Wheel.STL" />
-            </geometry>
-        </collision>
-    </link>
-    <link name="left_wheel_b">
-        <xacro:inertial_cylinder mass="0.1" length="0.01" radius="0.045">
-            <origin xyz="0 0 0" rpy="0 0 0"/>
-        </xacro:inertial_cylinder>
-        <visual>
-            <origin xyz="0 0 0" rpy="0 0 0" />
-            <geometry>
-                <mesh filename="file:///$(find ack_description)/meshes/Wheel.STL" />
-            </geometry>
-        </visual>
-        <collision>
-            <origin xyz="0 0 0" rpy="0 0 0" />
-            <geometry>
-                <mesh filename="file:///$(find ack_description)/meshes/Wheel.STL" />
-            </geometry>
-        </collision>
-    </link>
-    <link name="right_wheel_f">
-        <xacro:inertial_cylinder mass="0.1" length="0.01" radius="0.045">
-            <origin xyz="0 0 0" rpy="0 0 0"/>
-        </xacro:inertial_cylinder>
-        <visual>
-            <origin xyz="0 0 0" rpy="0 0 0" />
-            <geometry>
-                <mesh filename="file:///$(find ack_description)/meshes/Wheel.STL" />
-            </geometry>
-        </visual>
-        <collision>
-            <origin xyz="0 0 0" rpy="0 0 0" />
-            <geometry>
-                <mesh filename="file:///$(find ack_description)/meshes/Wheel.STL" />
-            </geometry>
-        </collision>
-    </link>
-    <link name="left_wheel_f">
-        <xacro:inertial_cylinder mass="0.1" length="0.01" radius="0.045">
-            <origin xyz="0 0 0" rpy="0 0 0"/>
-        </xacro:inertial_cylinder>
-        <visual>
-            <origin xyz="0 0 0" rpy="0 0 0" />
-            <geometry>
-                <mesh filename="file:///$(find ack_description)/meshes/Wheel.STL" />
-            </geometry>
-        </visual>
-        <collision>
-            <origin xyz="0 0 0" rpy="0 0 0" />
-            <geometry>
-                <mesh filename="file:///$(find ack_description)/meshes/Wheel.STL" />
-            </geometry>
-        </collision>
-    </link>
-    <link name="right_steer">
+    <link name="right_rear_wheel_link">
+        <xacro:inertial_cylinder mass="0.1" length="0.01" radius="0.045">
+            <origin xyz="0 0 0" rpy="0 0 0"/>
+        </xacro:inertial_cylinder>
+        <visual>
+            <origin xyz="0 0 0" rpy="0 0 0" />
+            <geometry>
+                <!-- <mesh filename="file:///$(find ack_description)/meshes/Wheel.STL" /> -->
+                <cylinder radius="0.045" length="0.01"/>
+                <material name="Black">
+                    <color rgba="0 0 0 1"/>
+                </material>
+            </geometry>
+        </visual>
+        <collision>
+            <origin xyz="0 0 0" rpy="0 0 0" />
+            <geometry>
+                <!-- <mesh filename="file:///$(find ack_description)/meshes/Wheel.STL" /> -->
+                <cylinder radius="0.045" length="0.01"/>
+            </geometry>
+        </collision>
+    </link>
+    <link name="left_rear_wheel_link">
+        <xacro:inertial_cylinder mass="0.1" length="0.01" radius="0.045">
+            <origin xyz="0 0 0" rpy="0 0 0"/>
+        </xacro:inertial_cylinder>
+        <visual>
+            <origin xyz="0 0 0" rpy="0 0 0" />
+            <geometry>
+                <!-- <mesh filename="file:///$(find ack_description)/meshes/Wheel.STL" /> -->
+                <cylinder radius="0.045" length="0.01"/>
+                <material name="Black">
+                    <color rgba="0 0 0 1"/>
+                </material>
+            </geometry>
+        </visual>
+        <collision>
+            <origin xyz="0 0 0" rpy="0 0 0" />
+            <geometry>
+                <!-- <mesh filename="file:///$(find ack_description)/meshes/Wheel.STL" /> -->
+                <cylinder radius="0.045" length="0.01"/>
+            </geometry>
+        </collision>
+    </link>
+    <link name="right_front_wheel_link">
+        <xacro:inertial_cylinder mass="0.1" length="0.01" radius="0.045">
+            <origin xyz="0 0 0" rpy="0 0 0"/>
+        </xacro:inertial_cylinder>
+        <visual>
+            <origin xyz="0 0 0" rpy="0 0 0" />
+            <geometry>
+                <!-- <mesh filename="file:///$(find ack_description)/meshes/Wheel.STL" /> -->
+                <cylinder radius="0.045" length="0.01"/>
+            </geometry>
+            <material name="Black">
+                <color rgba="0 0 0 1"/>
+            </material>
+        </visual>
+        <collision>
+            <origin xyz="0 0 0" rpy="0 0 0" />
+            <geometry>
+                <!-- <mesh filename="file:///$(find ack_description)/meshes/Wheel.STL" /> -->
+                <cylinder radius="0.045" length="0.01"/>
+            </geometry>
+        </collision>
+    </link>
+    <link name="left_front_wheel_link">
+        <xacro:inertial_cylinder mass="0.1" length="0.01" radius="0.045">
+            <origin xyz="0 0 0" rpy="0 0 0"/>
+        </xacro:inertial_cylinder>
+        <visual>
+            <origin xyz="0 0 0" rpy="0 0 0" />
+            <geometry>
+                <!-- <mesh filename="file:///$(find ack_description)/meshes/Wheel.STL" /> -->
+                <cylinder radius="0.045" length="0.01"/>
+                <material name="Black">
+                    <color rgba="0 0 0 1"/>
+                </material>
+            </geometry>
+        </visual>
+        <collision>
+            <origin xyz="0 0 0" rpy="0 0 0" />
+            <geometry>
+                <!-- <mesh filename="file:///$(find ack_description)/meshes/Wheel.STL" /> -->
+                <cylinder radius="0.045" length="0.01"/>
+            </geometry>
+        </collision>
+    </link>
+    <link name="right_steer_link">
         <xacro:inertial_flip_cylinder mass="0.1" length="0.01" radius="0.045">
             <origin xyz="0 0 0" rpy="0 0 0"/>
         </xacro:inertial_flip_cylinder>
     </link>
-    <link name="left_steer">
+    <link name="left_steer_link">
         <xacro:inertial_flip_cylinder mass="0.1" length="0.01" radius="0.045">
             <origin xyz="0 0 0" rpy="0 0 0"/>
@@ -109,32 +134,32 @@
     </link>
     <!-- WHEEL JOINT -->
-    <joint name="left_joint_b" type="continuous">
+    <joint name="left_rear_wheel" type="continuous">
         <origin xyz="-0.1 0.07 0" rpy="-1.57079632679 0 0" />
         <parent link="chassis" />
-        <child link="left_wheel_b" />
-        <axis xyz="0 0 1" />
-        <limit
-            effort="10.0"
-            lower="-3.14159265359"
-            upper="3.14159265359"
-            velocity="20.0"
-            />
-    </joint>
-    <joint name="right_joint_b" type="continuous">
+        <child link="left_rear_wheel_link" />
+        <axis xyz="0 0 1" />
+        <limit
+            effort="10.0"
+            lower="-3.14159265359"
+            upper="3.14159265359"
+            velocity="20.0"
+            />
+    </joint>
+    <joint name="right_rear_wheel" type="continuous">
         <origin xyz="-0.1 -0.07 0" rpy="-1.57079632679 0 0" />
         <parent link="chassis" />
-        <child link="right_wheel_b" />
-        <axis xyz="0 0 1" />
-        <limit
-            effort="10.0"
-            lower="-3.14159265359"
-            upper="3.14159265359"
-            velocity="20.0"
-            />
-    </joint>
-    <joint name="left_joint_s" type="revolute">
+        <child link="right_rear_wheel_link" />
+        <axis xyz="0 0 1" />
+        <limit
+            effort="10.0"
+            lower="-3.14159265359"
+            upper="3.14159265359"
+            velocity="20.0"
+            />
+    </joint>
+    <joint name="left_steer" type="revolute">
         <origin xyz="0.1 0.07 0" rpy="0 0 0" />
         <parent link="chassis" />
-        <child link="left_steer" />
+        <child link="left_steer_link" />
         <axis xyz="0 0 1" />
         <limit
@@ -144,20 +169,20 @@
             velocity="10.00"/>
     </joint>
-    <joint name="left_joint_f" type="continuous">
+    <joint name="left_front_wheel" type="continuous">
         <origin xyz="0 0 0" rpy="-1.57079632679 0 0" />
-        <parent link="left_steer" />
-        <child link="left_wheel_f" />
-        <axis xyz="0 0 1" />
-        <limit
-            effort="10.0"
-            lower="-3.14159265359"
-            upper="3.14159265359"
-            velocity="20.0"
-            />
-    </joint>
-    <joint name="right_joint_s" type="revolute">
+        <parent link="left_steer_link" />
+        <child link="left_front_wheel_link" />
+        <axis xyz="0 0 1" />
+        <limit
+            effort="10.0"
+            lower="-3.14159265359"
+            upper="3.14159265359"
+            velocity="20.0"
+            />
+    </joint>
+    <joint name="right_steer" type="revolute">
         <origin xyz="0.1 -0.07 0" rpy="0 0 0" />
         <parent link="chassis" />
-        <child link="right_steer" />
+        <child link="right_steer_link" />
         <axis xyz="0 0 1" />
         <limit
@@ -167,15 +192,22 @@
             velocity="10.00"/>
     </joint>
-    <joint name="right_joint_f" type="continuous">
+    <joint name="right_front_wheel" type="continuous">
         <origin xyz="0 0 0" rpy="-1.57079632679 0 0" />
-        <parent link="right_steer" />
-        <child link="right_wheel_f" />
-        <axis xyz="0 0 1" />
-        <limit
-            effort="10.0"
-            lower="-3.14159265359"
-            upper="3.14159265359"
-            velocity="20.0"
-            />
-    </joint>
+        <parent link="right_steer_link" />
+        <child link="right_front_wheel_link" />
+        <axis xyz="0 0 1" />
+        <limit
+            effort="10.0"
+            lower="-3.14159265359"
+            upper="3.14159265359"
+            velocity="20.0"
+            />
+    </joint>
+    <!-- TRANSMISSIONS -->
+    <xacro:wheel_transmission wheel_prefix="left_front"/>
+    <xacro:wheel_transmission wheel_prefix="right_front"/>
+    <xacro:wheel_transmission wheel_prefix="left_rear"/>
+    <xacro:wheel_transmission wheel_prefix="right_rear"/>
+    <xacro:steering_hinge_transmission wheel_prefix="left"/>
+    <xacro:steering_hinge_transmission wheel_prefix="right"/>
 </robot>

Commit message: edit gazebo add front wheel joints

File: src/ack_description/urdf/gazebo.xacro (robot description, xacro)
@@ -15,4 +15,20 @@
         </joint>
         <joint name="right_rear_wheel">
+            <command_interface name="velocity"/>
+            <state_interface name="position">
+                <param name="initial_value">0.0</param>
+            </state_interface>
+            <state_interface name="velocity"/>
+            <state_interface name="effort"/>
+        </joint>
+        <joint name="left_front_wheel">
+            <command_interface name="velocity"/>
+            <state_interface name="position">
+                <param name="initial_value">0.0</param>
+            </state_interface>
+            <state_interface name="velocity"/>S
+            <state_interface name="effort"/>
+        </joint>
+        <joint name="right_front_wheel">
             <command_interface name="velocity"/>
             <state_interface name="position">
