Commit message: Update Validate

File: src/ack_description/urdf/gazebo.xacro (robot description, xacro)
@@ -2,8 +2,23 @@
 <robot xmlns:xacro="http://www.ros.org/wiki/xacro" name="ackbot">
     <xacro:include filename="inertial_macros.xacro"/>
+    <xacro:include filename="transmission.xacro"/>
     <ros2_control name="GazeboSystem" type="system">
         <hardware>
             <plugin>gazebo_ros2_control/GazeboSystem</plugin>
         </hardware>
+        <joint name="left_front_wheel">
+            <state_interface name="position">
+                <param name="initial_value">0.0</param>
+            </state_interface>
+            <state_interface name="velocity"/>
+            <state_interface name="effort"/>
+        </joint>
+        <joint name="right_front_wheel">
+            <state_interface name="position">
+                <param name="initial_value">0.0</param>
+            </state_interface>
+            <state_interface name="velocity"/>
+            <state_interface name="effort"/>
+        </joint>
         <joint name="left_rear_wheel">
             <command_interface name="velocity"/>
@@ -22,20 +37,4 @@
             <state_interface name="effort"/>
         </joint>
-        <joint name="left_front_wheel">
-            <command_interface name="velocity"/>
-            <state_interface name="position">
-                <param name="initial_value">0.0</param>
-            </state_interface>
-            <state_interface name="velocity"/>S
-            <state_interface name="effort"/>
-        </joint>
-        <joint name="right_front_wheel">
-            <command_interface name="velocity"/>
-            <state_interface name="position">
-                <param name="initial_value">0.0</param>
-            </state_interface>
-            <state_interface name="velocity"/>
-            <state_interface name="effort"/>
-        </joint>
         <joint name="left_steer">
             <command_interface name="position">
@@ -43,5 +42,4 @@
                 <param name="max">0.60</param>
             </command_interface>
-            <command_interface name="velocity"/>
             <state_interface name="position">
                 <param name="initial_value">0.0</param>
@@ -55,5 +53,4 @@
                 <param name="max">0.60</param>
             </command_interface>
-            <command_interface name="velocity"/>
             <state_interface name="position">
                 <param name="initial_value">0.0</param>
@@ -62,4 +59,9 @@
             <state_interface name="effort"/>
         </joint>
+        <!-- TRANSMISSIONS -->
+        <xacro:wheel_transmission wheel_prefix="left_rear"/>
+        <xacro:wheel_transmission wheel_prefix="right_rear"/>
+        <xacro:steering_hinge_transmission wheel_prefix="left"/>
+        <xacro:steering_hinge_transmission wheel_prefix="right"/>
     </ros2_control>
     <gazebo>
@@ -80,14 +82,10 @@
       </plugin>
     </gazebo>
-    <!-- <gazebo>
-        <plugin name="gazebo_ros_joint_state_publisher" filename="libgazebo_ros_joint_state_publisher.so">
-            <always_on>true</always_on>
-            <update_rate>100.0</update_rate>
-        </plugin>
-    </gazebo> -->
     <gazebo reference="chassis">
         <mu1>0.2</mu1>
         <mu2>0.2</mu2>
         <material>Gazebo/Red</material>
+        <kp  value="10000000.0"/>
+        <kd value="0.2"/>
     </gazebo>
     <gazebo reference="left_steer_link">
@@ -95,4 +93,6 @@
         <mu2>0.2</mu2>
         <material>Gazebo/Red</material>
+        <kp  value="10000000.0"/>
+        <kd value="0.2"/>
     </gazebo>
     <gazebo reference="right_steer_link">
@@ -100,4 +100,6 @@
         <mu2>0.2</mu2>
         <material>Gazebo/Red</material>
+        <kp  value="10000000.0"/>
+        <kd value="0.2"/>
     </gazebo>
     <gazebo reference="left_front_wheel_link">
@@ -105,4 +107,6 @@
         <mu2>0.2</mu2>
         <material>Gazebo/Black</material>
+        <kp  value="10000000.0"/>
+        <kd value="0.2"/>
     </gazebo>
     <gazebo reference="left_rear_wheel_link">
@@ -110,4 +114,6 @@
         <mu2>0.2</mu2>
         <material>Gazebo/Black</material>
+        <kp  value="10000000.0"/>
+        <kd value="0.2"/>
     </gazebo>
     <gazebo reference="right_front_wheel_link">
@@ -115,4 +121,6 @@
         <mu2>0.2</mu2>
         <material>Gazebo/Black</material>
+        <kp  value="10000000.0"/>
+        <kd value="0.2"/>
     </gazebo>
     <gazebo reference="right_rear_wheel_link">
@@ -120,4 +128,6 @@
         <mu2>0.2</mu2>
         <material>Gazebo/Black</material>
+        <kp  value="10000000.0"/>
+        <kd value="0.2"/>
     </gazebo>
 </robot>

File: src/ack_description/urdf/robot.xacro (robot description, xacro)
@@ -3,5 +3,4 @@
     <xacro:include filename="gazebo.xacro"/>
     <xacro:include filename="imu.xacro"/>
-    <xacro:include filename="transmission.xacro"/>
     <!-- BASE LINK -->
     <link name="base_link">
@@ -20,5 +19,4 @@
             <origin xyz="0 0 0.025" rpy="0 0 0" />
             <geometry>
-                <!-- <mesh filename="file:///$(find ack_description)/meshes/Body.STL"/> -->
                 <box size="0.2 0.13 0.05"/>
             </geometry>
@@ -42,5 +40,4 @@
             <origin xyz="0 0 0" rpy="0 0 0" />
             <geometry>
-                <!-- <mesh filename="file:///$(find ack_description)/meshes/Wheel.STL" /> -->
                 <cylinder radius="0.045" length="0.01"/>
                 <material name="Black">
@@ -52,5 +49,4 @@
             <origin xyz="0 0 0" rpy="0 0 0" />
             <geometry>
-                <!-- <mesh filename="file:///$(find ack_description)/meshes/Wheel.STL" /> -->
                 <cylinder radius="0.045" length="0.01"/>
             </geometry>
@@ -64,5 +60,4 @@
             <origin xyz="0 0 0" rpy="0 0 0" />
             <geometry>
-                <!-- <mesh filename="file:///$(find ack_description)/meshes/Wheel.STL" /> -->
                 <cylinder radius="0.045" length="0.01"/>
                 <material name="Black">
@@ -74,5 +69,4 @@
             <origin xyz="0 0 0" rpy="0 0 0" />
             <geometry>
-                <!-- <mesh filename="file:///$(find ack_description)/meshes/Wheel.STL" /> -->
                 <cylinder radius="0.045" length="0.01"/>
             </geometry>
@@ -86,5 +80,4 @@
             <origin xyz="0 0 0" rpy="0 0 0" />
             <geometry>
-                <!-- <mesh filename="file:///$(find ack_description)/meshes/Wheel.STL" /> -->
                 <cylinder radius="0.045" length="0.01"/>
             </geometry>
@@ -96,5 +89,4 @@
             <origin xyz="0 0 0" rpy="0 0 0" />
             <geometry>
-                <!-- <mesh filename="file:///$(find ack_description)/meshes/Wheel.STL" /> -->
                 <cylinder radius="0.045" length="0.01"/>
             </geometry>
@@ -108,5 +100,4 @@
             <origin xyz="0 0 0" rpy="0 0 0" />
             <geometry>
-                <!-- <mesh filename="file:///$(find ack_description)/meshes/Wheel.STL" /> -->
                 <cylinder radius="0.045" length="0.01"/>
                 <material name="Black">
@@ -118,5 +109,4 @@
             <origin xyz="0 0 0" rpy="0 0 0" />
             <geometry>
-                <!-- <mesh filename="file:///$(find ack_description)/meshes/Wheel.STL" /> -->
                 <cylinder radius="0.045" length="0.01"/>
             </geometry>
@@ -204,10 +194,3 @@
             />
     </joint>
-    <!-- TRANSMISSIONS -->
-    <xacro:wheel_transmission wheel_prefix="left_front"/>
-    <xacro:wheel_transmission wheel_prefix="right_front"/>
-    <xacro:wheel_transmission wheel_prefix="left_rear"/>
-    <xacro:wheel_transmission wheel_prefix="right_rear"/>
-    <xacro:steering_hinge_transmission wheel_prefix="left"/>
-    <xacro:steering_hinge_transmission wheel_prefix="right"/>
 </robot>

File: src/ack_description/urdf/transmission.xacro (robot description, xacro)
@@ -2,24 +2,26 @@
 <robot name="ackbot" xmlns:xacro="http://ros.org/wiki/xacro">
     <xacro:macro name="wheel_transmission" params="wheel_prefix">
-        <transmission name="${wheel_prefix}_wheel_trans" type="SimpleTransmission">
-            <type>transmission_interface/SimpleTransmission</type>
-            <actuator name="${wheel_prefix}_wheel_motor">
-                <hardwareInterface>hardware_interface/VelocityJointInterface</hardwareInterface>
+        <transmission name="${wheel_prefix}_wheel_trans">
+        <plugin>transmission_interface/SimpleTransmission</plugin>
+            <!-- <type>transmission_interface/SimpleTransmission</type> -->
+            <actuator name="${wheel_prefix}_wheel_motor" role="${wheel_prefix}_wheel_motor">
+                <hardwareInterface>VelocityJointInterface</hardwareInterface>
+            </actuator>
+            <joint name="${wheel_prefix}_wheel" role="{wheel_prefix}_wheel">
+                <hardwareInterface>VelocityJointInterface</hardwareInterface>
                 <mechanicalReduction>1</mechanicalReduction>
-            </actuator>
-            <joint name="${wheel_prefix}_wheel">
-                <hardwareInterface>hardware_interface/VelocityJointInterface</hardwareInterface>
             </joint>
         </transmission>
     </xacro:macro>
     <xacro:macro name="steering_hinge_transmission" params="wheel_prefix">
-        <transmission name="${wheel_prefix}_wheel_trans" type="SimpleTransmission">
-            <type>transmission_interface/SimpleTransmission</type>
-            <actuator name="${wheel_prefix}_wheel_motor">
-                <hardwareInterface>hardware_interface/PositionJointInterface</hardwareInterface>
+        <transmission name="${wheel_prefix}_wheel_trans">
+        <plugin>transmission_interface/SimpleTransmission</plugin>
+            <!-- <type>transmission_interface/SimpleTransmission</type> -->
+            <actuator name="${wheel_prefix}_steer_motor" role="${wheel_prefix}_steer_motor">
+                <hardwareInterface>PositionJointInterface</hardwareInterface>
+            </actuator>
+            <joint name="${wheel_prefix}_steer" role="${wheel_prefix}_steer">
+                <hardwareInterface>PositionJointInterface</hardwareInterface>
                 <mechanicalReduction>1</mechanicalReduction>
-            </actuator>
-            <joint name="${wheel_prefix}_wheel">
-                <hardwareInterface>hardware_interface/PositionJointInterface</hardwareInterface>
             </joint>
         </transmission>
